Commit message: commit

File: hexapod_gazebo_description/urdf/hexapod_gazebo.xacro (robot description, xacro)
@@ -2,22 +2,26 @@
 <robot xmlns:xacro="http://www.ros.org/wiki/xacro" name="hexapod">
   <xacro:property name="M_PI" value="3.1415926535897931"/>
+  <xacro:property name="gen3" value="1.7320508075689"/>
   <xacro:property name="bodyradius" value="0.1800"/>
   <xacro:property name="bodylength" value="0.1000"/>
   <xacro:property name="bodymass" value="3"/>
   <xacro:property name="bridgelength" value="0.01"/>
-  <xacro:property name="bridgeradius" value="0.02"/>
+  <xacro:property name="bridgeradius" value="0.03"/>
   <xacro:property name="bridgemass" value="0.5"/>
-  <xacro:property name="rolllength" value="0.14489"/>
+  <xacro:property name="rolllength" value="0.093"/>
   <xacro:property name="rollradius" value="0.03"/>
   <xacro:property name="rollmass" value="${rolllength*5}"/>
-  <xacro:property name="pitch1length" value="0.164"/>
+  <xacro:property name="pitch1length" value="0.14489"/>
   <xacro:property name="pitch1radius" value="0.03"/>
   <xacro:property name="pitch1mass" value="${pitch1length*5}"/>
-  <xacro:property name="pitch2length" value="0.157"/>
+  <xacro:property name="pitch2length" value="0.164"/>
   <xacro:property name="pitch2radius" value="0.03"/>
   <xacro:property name="pitch2mass" value="${pitch2length*5}"/>
+  <xacro:property name="pitch3length" value="0.157"/>
+  <xacro:property name="pitch3radius" value="0.03"/>
+  <xacro:property name="pitch3mass" value="${pitch3length*5}"/>
   <xacro:property name="sticklength" value="0.01"/>
-  <xacro:property name="stickradius" value="0.08"/>
-  <xacro:property name="stickmass" value="0.5"/>
+  <xacro:property name="stickradius" value="0.1"/>
+  <xacro:property name="stickmass" value="1"/>
   <xacro:property name="damping" value="1"/>
 <link name="base_link">
@@ -37,6 +41,6 @@
      <cylinder length="${bodylength}" radius="${bodyradius}"/>
    </geometry>
-   <material name="black">
-     <color rgba="0 0 0 100"/>
+   <material name="Red">
+     <color rgba="255 0 0 100"/>
    </material>
   </visual>
@@ -68,14 +72,14 @@
 <link name="${leg}_bridge">
   <visual>
-    <origin xyz="0 0 ${bridgelength/2}" rpy="0 0 0"/>
+    <origin xyz="${bridgelength/2} 0 0" rpy="0 ${M_PI/2} 0"/>
     <geometry>
       <cylinder length="${bridgelength}" radius="${bridgeradius}"/>
     </geometry>
-    <material name="white">
-      <color rgba="255 255 255 1"/>
+    <material name="Black">
+      <color rgba="0 0 0 1"/>
     </material>
   </visual>
   <inertial>
-      <origin xyz="0 0 ${bridgelength/2}" rpy="0 0 0"/>
+    <origin xyz="0 0 0" rpy="0 0 0"/>
       <mass value="${bridgemass}"/>
       <inertia
@@ -85,5 +89,5 @@
     </inertial>
   <collision>
-    <origin xyz="0 0 ${bridgelength/2}" rpy="0 0 0"/>
+    <origin xyz="${bridgelength/2} 0 0" rpy="0 ${M_PI/2} 0"/>
     <geometry>
       <cylinder length="${bridgelength}" radius="${bridgeradius}"/>
@@ -102,14 +106,14 @@
 <link name="${leg}_roll">
   <visual>
-    <origin xyz="0 0 ${rolllength/2}" rpy="0 0 0"/>
+    <origin xyz="${rolllength/2} 0 0" rpy="0 ${M_PI/2} 0"/>
     <geometry>
       <cylinder length="${rolllength}" radius="${rollradius}"/>
     </geometry>
-    <material name="blue">
-      <color rgba="0 0 255 1"/>
+    <material name="Black">
+      <color rgba="0 0 0 1"/>
     </material>
   </visual>
   <inertial>
-    <origin xyz="0 0 ${rolllength/2}" rpy="0 0 0"/>
+    <origin xyz="0 0 0" rpy="0 0 0"/>
       <mass value="${rollmass}"/>
       <inertia
@@ -119,5 +123,5 @@
     </inertial>
   <collision>
-    <origin xyz="0 0 ${rolllength/2}" rpy="0 0 0"/>
+    <origin xyz="${rolllength/2} 0 0" rpy="0 ${M_PI/2} 0"/>
     <geometry>
       <cylinder length="${rolllength}" radius="${rollradius}"/>
@@ -129,31 +133,31 @@
   </gazebo>
 <joint name="${leg}_roll" type="revolute">
-  <axis xyz="1 0 0"/>
-  <limit effort="300" lower="-${M_PI/2}" upper="${M_PI/2}" velocity="1"/>
+  <axis xyz="0 0 1"/>
+  <limit effort="300" lower="-${M_PI/4}" upper="${M_PI/4}" velocity="1"/>
   <dynamics damping="${damping}"/>
   <parent link="${leg}_bridge"/>
   <child link="${leg}_roll"/>
-  <origin rpy="0 0 0" xyz="0 0 ${bridgelength}"/>
+  <origin rpy="0 0 0" xyz="0 0 0"/>
 </joint>
 <link name="${leg}_pitch1">
   <visual>
-    <origin xyz="0 0 ${pitch1length/2}" rpy="0 0 0"/>
+    <origin xyz="${pitch1length/2} 0 0" rpy="0 ${M_PI/2} 0"/>
     <geometry>
       <cylinder length="${pitch1length}" radius="${pitch1radius}"/>
     </geometry>
-    <material name="green">
-      <color rgba="0 128 0 1"/>
-    </material>
-  </visual>
- <inertial>
-    <origin xyz="0 0 ${pitch1length/2}" rpy="0 0 0"/>
+    <material name="Red">
+      <color rgba="255 0 0 1"/>
+    </material>
+  </visual>
+ <inertial>
+    <origin xyz="0 0 0" rpy="0 0 0"/>
       <mass value="${pitch1mass}"/>
       <inertia
-        ixx="${(3*pitch1mass*pitch1radius*pitch1radius+4*pitch1mass*pitch1length*pitch1length)/12}" ixy="0.0" ixz="0.0"
-        iyy="${0.5*pitch1mass*pitch1radius*pitch1radius}" iyz="0.0"
+        ixx="${0.5*pitch1mass*pitch1radius*pitch1radius}" ixy="0.0" ixz="0.0"
+        iyy="${(3*pitch1mass*pitch1radius*pitch1radius+4*pitch1mass*pitch1length*pitch1length)/12}" iyz="0.0"
         izz="${(3*pitch1mass*pitch1radius*pitch1radius+4*pitch1mass*pitch1length*pitch1length)/12}"/>
     </inertial>
   <collision>
-    <origin xyz="0 0 ${pitch1length/2}" rpy="0 0 0"/>
+    <origin xyz="${pitch1length/2} 0 0" rpy="0 ${M_PI/2} 0"/>
     <geometry>
       <cylinder length="${pitch1length}" radius="${pitch1radius}"/>
@@ -165,14 +169,14 @@
   </gazebo>
 <joint name="${leg}_pitch1" type="revolute">
-  <axis xyz="0 1 0"/>
-  <limit effort="300" lower="-${M_PI/2}" upper="${M_PI/2}" velocity="1"/>
+  <axis xyz="0 0 1"/>
+  <limit effort="300" lower="-${M_PI/3*2}" upper="${M_PI/2}" velocity="1"/>
   <dynamics damping="${damping}"/>
   <parent link="${leg}_roll"/>
   <child link="${leg}_pitch1"/>
-  <origin rpy="0 0 0" xyz="0 0 ${rolllength}"/>
+  <origin rpy="${M_PI/2} 0 0" xyz="${rolllength} 0 0"/>
 </joint>
 <link name="${leg}_pitch2">
   <visual>
-    <origin xyz="0 0 ${pitch2length/2}" rpy="0 0 0"/>
+    <origin xyz="${pitch2length/2} 0 0" rpy="${M_PI/2} 0 ${M_PI/2}"/>
     <geometry>
       <cylinder length="${pitch2length}" radius="${pitch2radius}"/>
@@ -183,13 +187,13 @@
   </visual>
  <inertial>
-    <origin xyz="0 0 ${pitch2length/2}" rpy="0 0 0"/>
+    <origin xyz="${pitch2length} 0 0" rpy="0 0 0"/>
       <mass value="${pitch2mass}"/>
       <inertia
-        ixx="${(3*pitch2mass*pitch2radius*pitch2radius+4*pitch2mass*pitch2length*pitch2length)/12}" ixy="0.0" ixz="0.0"
-        iyy="${0.5*pitch2mass*pitch2radius*pitch2radius}" iyz="0.0"
+        ixx="${0.5*pitch2mass*pitch2radius*pitch2radius}" ixy="0.0" ixz="0.0"
+        iyy="${(3*pitch2mass*pitch2radius*pitch2radius+4*pitch2mass*pitch2length*pitch2length)/12}" iyz="0.0"
         izz="${(3*pitch2mass*pitch2radius*pitch2radius+4*pitch2mass*pitch2length*pitch2length)/12}"/>
     </inertial>
   <collision>
-    <origin xyz="0 0 ${pitch2length/2}" rpy="0 0 0"/>
+    <origin xyz="${pitch2length/2} 0 0" rpy="${M_PI/2} 0 ${M_PI/2}"/>
     <geometry>
       <cylinder length="${pitch2length}" radius="${pitch2radius}"/>
@@ -203,10 +207,48 @@
   </gazebo>
 <joint name="${leg}_pitch2" type="revolute">
-  <axis xyz="0 1 0"/>
-  <limit effort="300" lower="-${M_PI/2}" upper="${M_PI/3}" velocity="1"/>
+  <axis xyz="0 0 1"/>
+  <limit effort="300" lower="-${M_PI/3}" upper="${M_PI/2}" velocity="1"/>
   <dynamics damping="${damping}"/>
   <parent link="${leg}_pitch1"/>
   <child link="${leg}_pitch2"/>
-  <origin rpy="0 ${M_PI/2} 0" xyz="0 0 ${pitch1length}"/>
+  <origin rpy="0 0 -${M_PI/2}" xyz="${pitch1length} 0 0"/>
+</joint>
+<link name="${leg}_pitch3">
+  <visual>
+    <origin xyz="${pitch3length/2} 0 0" rpy="${M_PI/2} 0 ${M_PI/2}"/>
+    <geometry>
+      <cylinder length="${pitch3length}" radius="${pitch3radius}"/>
+    </geometry>
+    <material name="Red">
+      <color rgba="255 0 0 1"/>
+    </material>
+  </visual>
+ <inertial>
+    <origin xyz="0 0 0" rpy="0 0 0"/>
+      <mass value="${pitch3mass}"/>
+      <inertia
+        ixx="${0.5*pitch3mass*pitch3radius*pitch3radius}" ixy="0.0" ixz="0.0"
+        iyy="${(3*pitch3mass*pitch3radius*pitch3radius+4*pitch3mass*pitch3length*pitch3length)/12}" iyz="0.0"
+        izz="${(3*pitch3mass*pitch3radius*pitch3radius+4*pitch3mass*pitch3length*pitch3length)/12}"/>
+    </inertial>
+  <collision>
+    <origin xyz="${pitch3length/2} 0 0" rpy="${M_PI/2} 0 ${M_PI/2}"/>
+    <geometry>
+      <cylinder length="${pitch3length}" radius="${pitch3radius}"/>
+    </geometry>
+  </collision>
+</link>
+  <gazebo reference="${leg}_pitch3">
+    <material>Gazebo/Red</material>
+    <mu1 value="200"/>
+    <mu2 value="200"/>
+  </gazebo>
+<joint name="${leg}_pitch3" type="revolute">
+  <axis xyz="0 0 1"/>
+  <limit effort="300" lower="-${M_PI/3}" upper="${M_PI/2}" velocity="1"/>
+  <dynamics damping="${damping}"/>
+  <parent link="${leg}_pitch2"/>
+  <child link="${leg}_pitch3"/>
+  <origin rpy="0 0 0" xyz="${pitch2length} 0 0"/>
 </joint>
 <!--stick-->
@@ -215,5 +257,5 @@
     <origin xyz="0 0 0" rpy="0 0 0"/>
     <geometry>
-      <cylinder length="0.001" radius="0.001"/>
+      <cylinder length="0.01" radius="0.01"/>
     </geometry>
     <material name="yellow">
@@ -222,5 +264,5 @@
   </visual>
  <inertial>
-    <origin xyz="0 0 ${pitch2length+sticklength}" rpy="0 0 0"/>
+    <origin xyz="0 0 0" rpy="0 0 0"/>
       <mass value="${stickmass}"/>
       <inertia
@@ -232,33 +274,33 @@
     <origin xyz="0 0 0" rpy="0 0 0"/>
     <geometry>
-      <cylinder length="0.001" radius="0.001"/>
+      <cylinder length="0.01" radius="0.01"/>
     </geometry>
   </collision>
 </link>
 <joint name="${leg}_stick1" type="revolute">
-  <limit effort="300" lower="-${M_PI/2}" upper="${M_PI/2}" velocity="1"/>
+  <limit effort="300" lower="-${M_PI/7}" upper="${M_PI/7}" velocity="1"/>
   <dynamics damping="${damping}"/>
   <axis xyz="1 0 0"/>
-  <parent link="${leg}_pitch2"/>
+  <parent link="${leg}_pitch3"/>
   <child link="${leg}_stick1"/>
-  <origin rpy="0 0 0" xyz="0 0 ${pitch2length+sticklength}"/>
+  <origin rpy="0 ${M_PI/2} 0" xyz="${pitch2length+sticklength/2} 0 0"/>
 </joint>
   <gazebo reference="${leg}_stick1">
     <material>Gazebo/Black</material>
-    <mu1 value="10"/>
-    <mu2 value="10"/>
-  </gazebo>
-<link name="${leg}_stick2">
-  <visual>
-    <origin xyz="0 0 0" rpy="0 0 0"/>
-    <geometry>
-      <cylinder length="0.001" radius="0.001"/>
-    </geometry>
-    <material name="yellow">
-      <color rgba="255 255 0 1"/>
-    </material>
-  </visual>
- <inertial>
-    <origin xyz="0 0 ${pitch2length+sticklength}" rpy="0 0 0"/>
+    <mu1 value="10000"/>
+    <mu2 value="10000"/>
+  </gazebo>
+<link name="${leg}_stick3">
+  <visual>
+    <origin xyz="0 0 0" rpy="0 0 0"/>
+    <geometry>
+      <cylinder length="${sticklength}" radius="${stickradius}"/>
+    </geometry>
+    <material name="Black">
+      <color rgba="0 0 0 1"/>
+    </material>
+  </visual>
+ <inertial>
+    <origin xyz="0 0 0" rpy="0 0 0"/>
       <mass value="${stickmass}"/>
       <inertia
@@ -270,22 +312,22 @@
     <origin xyz="0 0 0" rpy="0 0 0"/>
     <geometry>
-      <cylinder length="0.001" radius="0.001"/>
-    </geometry>
-  </collision>
-</link>
-<joint name="${leg}_stick2" type="revolute">
-  <limit effort="300" lower="-${M_PI/2}" upper="${M_PI/2}" velocity="1"/>
+      <cylinder length="${sticklength}" radius="${stickradius}"/>
+    </geometry>
+  </collision>
+</link>
+<joint name="${leg}_stick3" type="revolute">
+  <limit effort="300" lower="-${M_PI/7}" upper="${M_PI/7}" velocity="1"/>
   <dynamics damping="${damping}"/>
   <axis xyz="0 1 0"/>
   <parent link="${leg}_stick1"/>
-  <child link="${leg}_stick2"/>
+  <child link="${leg}_stick3"/>
   <origin rpy="0 0 0" xyz="0 0 0"/>
 </joint>
-  <gazebo reference="${leg}_stick2">
-    <material>Gazebo/Black</material>
-    <mu1 value="10"/>
-    <mu2 value="10"/>
-  </gazebo>
-<link name="${leg}_stick3">
+  <gazebo reference="${leg}_stick3">
+    <material>Gazebo/Black</material>
+    <mu1 value="10000"/>
+    <mu2 value="10000"/>
+  </gazebo>
+<!--<link name="${leg}_stick3">
   <visual>
     <origin xyz="0 0 0" rpy="0 0 0"/>
@@ -293,10 +335,10 @@
       <cylinder length="${sticklength}" radius="${stickradius}"/>
     </geometry>
-    <material name="yellow">
-      <color rgba="255 255 0 1"/>
-    </material>
-  </visual>
- <inertial>
-    <origin xyz="0 0 ${pitch2length+sticklength}" rpy="0 0 0"/>
+    <material name="Black">
+      <color rgba="0 0 0 1"/>
+    </material>
+  </visual>
+ <inertial>
+    <origin xyz="0 0 0" rpy="0 0 0"/>
       <mass value="${stickmass}"/>
       <inertia
@@ -313,7 +355,7 @@
 </link>
 <joint name="${leg}_stick3" type="revolute">
-  <limit effort="300" lower="-${M_PI/2}" upper="${M_PI/2}" velocity="1"/>
-  <dynamics damping="${damping}"/>
-  <axis xyz="0 0 1"/>
+  <limit effort="300" lower="-${M_PI/7}" upper="${M_PI/7}" velocity="1"/>
+  <dynamics damping="${damping}"/>
+  <axis xyz="0 1 0"/>
   <parent link="${leg}_stick2"/>
   <child link="${leg}_stick3"/>
@@ -322,43 +364,8 @@
   <gazebo reference="${leg}_stick3">
     <material>Gazebo/Black</material>
-    <mu1 value="2000"/>
-    <mu2 value="2000"/>
-  </gazebo>
-<!--<link name="${leg}_stick">
-  <visual>
-    <origin xyz="0 0 ${pitch2length+sticklength}" rpy="0 0 0"/>
-    <geometry>
-      <cylinder length="${sticklength}" radius="${stickradius}"/>
-    </geometry>
-    <material name="yellow">
-      <color rgba="255 255 0 1"/>
-    </material>
-  </visual>
- <inertial>
-    <origin xyz="0 0 ${pitch2length+sticklength}" rpy="0 0 0"/>
-      <mass value="${stickmass}"/>
-      <inertia
-        ixx="${(3*stickmass*stickradius*stickradius+4*stickmass*sticklength*sticklength)/12}" ixy="0.0" ixz="0.0"
-        iyy="${(3*stickmass*stickradius*stickradius+4*stickmass*sticklength*sticklength)/12}" iyz="0.0"
-        izz="${0.5*stickmass*stickradius*stickradius}"/>
-    </inertial>
-  <collision>
-    <origin xyz="0 0 ${pitch2length+sticklength}" rpy="0 0 0"/>
-    <geometry>
-      <cylinder length="${sticklength}" radius="${stickradius}"/>
-    </geometry>
-  </collision>
-</link>
-<joint name="${leg}_stick" type="fixed">
-  <axis xyz="0 0 1"/>
-  <parent link="${leg}_pitch2"/>
-  <child link="${leg}_stick"/>
-  <origin rpy="0 0 0" xyz="0 0 0"/>
-</joint>
-  <gazebo reference="${leg}_stick">
-    <material>Gazebo/Black</material>
-    <mu1 value="10"/>
-    <mu2 value="10"/>
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
Commit message: 角度平滑，舍弃线性插值

File: hexapod_gazebo_description/urdf/hexapod_gazebo.xacro (robot description, xacro)
@@ -22,5 +22,5 @@
   <xacro:property name="pitch3mass" value="${pitch3length*5}"/>
   <xacro:property name="sticklength" value="0.01"/>
-  <xacro:property name="stickradius" value="0.1"/>
+  <xacro:property name="stickradius" value="0.07"/>
   <xacro:property name="stickmass" value="1"/>
   <xacro:property name="damping" value="1"/>
@@ -134,5 +134,5 @@
 <joint name="${leg}_roll" type="revolute">
   <axis xyz="0 0 1"/>
-  <limit effort="300" lower="-${M_PI/4}" upper="${M_PI/4}" velocity="1"/>
+  <limit effort="300" lower="-${M_PI/2}" upper="${M_PI/2}" velocity="1"/>
   <dynamics damping="${damping}"/>
   <parent link="${leg}_bridge"/>
@@ -170,5 +170,5 @@
 <joint name="${leg}_pitch1" type="revolute">
   <axis xyz="0 0 1"/>
-  <limit effort="300" lower="-${M_PI/3*2}" upper="${M_PI/2}" velocity="1"/>
+  <limit effort="300" lower="-${M_PI/2*3}" upper="${M_PI/2}" velocity="1"/>
   <dynamics damping="${damping}"/>
   <parent link="${leg}_roll"/>
@@ -208,5 +208,5 @@
 <joint name="${leg}_pitch2" type="revolute">
   <axis xyz="0 0 1"/>
-  <limit effort="300" lower="-${M_PI/3}" upper="${M_PI/2}" velocity="1"/>
+  <limit effort="300" lower="-${M_PI*2/3}" upper="${M_PI}" velocity="1"/>
   <dynamics damping="${damping}"/>
   <parent link="${leg}_pitch1"/>
@@ -246,5 +246,5 @@
 <joint name="${leg}_pitch3" type="revolute">
   <axis xyz="0 0 1"/>
-  <limit effort="300" lower="-${M_PI/3}" upper="${M_PI/2}" velocity="1"/>
+  <limit effort="300" lower="-${M_PI*2/3}" upper="${M_PI/2}" velocity="1"/>
   <dynamics damping="${damping}"/>
   <parent link="${leg}_pitch2"/>
@@ -279,5 +279,5 @@
 </link>
 <joint name="${leg}_stick1" type="revolute">
-  <limit effort="300" lower="-${M_PI/7}" upper="${M_PI/7}" velocity="1"/>
+  <limit effort="300" lower="-${M_PI/180}" upper="${M_PI/180}" velocity="1"/>
   <dynamics damping="${damping}"/>
   <axis xyz="1 0 0"/>
@@ -317,5 +317,5 @@
 </link>
 <joint name="${leg}_stick3" type="revolute">
-  <limit effort="300" lower="-${M_PI/7}" upper="${M_PI/7}" velocity="1"/>
+  <limit effort="300" lower="-${M_PI/180}" upper="${M_PI/180}" velocity="1"/>
   <dynamics damping="${damping}"/>
   <axis xyz="0 1 0"/>
@@ -355,5 +355,5 @@
 </link>
 <joint name="${leg}_stick3" type="revolute">
-  <limit effort="300" lower="-${M_PI/7}" upper="${M_PI/7}" velocity="1"/>
+  <limit effort="300" lower="-${M_PI/60}" upper="${M_PI/60}" velocity="1"/>
   <dynamics damping="${damping}"/>
   <axis xyz="0 1 0"/>

Commit message: rviz同步显示

File: hexapod_gazebo_description/urdf/hexapod_gazebo.xacro (robot description, xacro)
@@ -67,5 +67,5 @@
   <parent link="base_link"/>
   <child link="body"/>
-  <origin rpy="0 0 0" xyz="0 0 0"/>
+  <origin rpy="0 0 0" xyz="0 0 ${pitch2length+pitch3length+sticklength}"/>
 </joint>
   <xacro:macro name="leg" params="leg r p ry x y">
